File: recorder/recorder.kicad_pcb (KiCad board)
At the start: 2 copper layers, 34 parts, among them J1 GPIO_Conn_02x20_Odd_Even, U1 IM73D122V01, U10 TPS7A4700RGWT, U2 ADAU7118, U3 IM73D122V01, U4 IM73D122V01, U5 IM73D122V01, U6 IM73D122V01, U7 IM73D122V01, U8 IM73D122V01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

Commit message: v0
Parts:
- moved U4 119.7 mm to (300.5, 314.5)
- moved U5 119.7 mm to (385.5, 314.5)
- moved U6 119.7 mm to (470.5, 314.5)
- moved U7 119.7 mm to (555.5, 314.5)
- moved U8 119.7 mm to (640.5, 314.5)
- moved U9 119.7 mm to (725.5, 314.5)
- moved U1 119.7 mm to (130.5, 314.5)
- moved U3 119.7 mm to (215.5, 314.5)
- moved C1 114.2 mm to (130.8, 311.0), turned to 180 degrees
- moved C2 114.2 mm to (215.8, 311.0), turned to 180 degrees
- moved C3 114.2 mm to (300.8, 311.0), turned to 180 degrees
- moved C4 114.1 mm to (385.7, 311.0), turned to 180 degrees
- moved C5 114.1 mm to (470.7, 311.0), turned to 180 degrees
- moved C6 114.1 mm to (555.7, 311.0), turned to 180 degrees
- moved C7 114.1 mm to (640.7, 311.0), turned to 180 degrees
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
Commit message: ground planes
Parts:
- moved J1 75.2 mm to (338.1, 301.0)
- moved C11 57.3 mm to (448.6, 297.0), turned to 0 degrees
- moved U2 57.1 mm to (449.5, 300.2), turned to 90 degrees
- moved C9 51.9 mm to (446.4, 298.7), turned to 90 degrees
- moved C10 50.2 mm to (446.4, 302.0), turned to -90 degrees
- moved R9 48.1 mm to (444.9, 300.3), turned to -90 degrees
- moved C13 41.2 mm to (439.1, 296.0), turned to 180 degrees
- moved C12 40.1 mm to (441.6, 304.0), turned to 180 degrees
- moved U10 39.2 mm to (440.0, 300.0), turned to -90 degrees
- moved C14 34.2 mm to (438.6, 304.0), turned to 180 degrees
- moved R6 25.1 mm to (573.2, 297.0)
- moved R7 25.1 mm to (658.2, 297.0)
- moved R4 25.1 mm to (403.2, 297.0)
- moved R1 25.1 mm to (148.2, 297.0)
- moved C4 24.9 mm to (406.3, 297.0)
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Routing:
- added copper zone on In2.Cu, net /DVDD
- added copper zone on In1.Cu, net GND
Other:
- copper layers 2 -> 4

Commit message: pre crash
Routing:
- net /DAT1: track 0.00 -> 613.7 mm
- net /DAT0: track 0.00 -> 611.2 mm

Commit message: traces man traces
Parts:
- moved J1 169.7 mm to (507.8, 299.0)
Routing:
- net /DAT3: track 0.00 -> 339.1 mm
- net /DAT0: track 611.2 -> 351.0 mm
- net /DAT1: track 613.7 -> 386.4 mm
- net /DAT2: track 0.00 -> 169.9 mm

Commit message: Re-routed, removed signal lines, set the CLK lines as priority.
Parts:
- moved J1 85.5 mm to (422.8, 290.0)
Routing:
- net /CLK0: track 0.00 -> 520.6 mm
- net /CLK1: track 0.00 -> 515.6 mm
- net /DAT1: track 386.4 -> 0.00 mm
- net /DAT0: track 351.0 -> 0.00 mm
- net /DAT3: track 339.1 -> 0.00 mm
- net /DAT2: track 169.9 -> 0.00 mm
- net /DVDD: track 0.00 -> 28.9 mm
- net Net-(U3-DATA): track 0.00 -> 2.86 mm
- net Net-(U9-DATA): track 0.00 -> 2.86 mm
- net Net-(U6-DATA): track 0.00 -> 2.86 mm
- net Net-(U4-DATA): track 0.00 -> 2.86 mm
- net Net-(U8-DATA): track 0.00 -> 2.86 mm
- net Net-(U7-DATA): track 0.00 -> 2.86 mm
- net Net-(U5-DATA): track 0.00 -> 2.86 mm
- net Net-(U1-DATA): track 0.00 -> 2.86 mm

Commit message: data 0 routed
Parts:
- moved C11 1.29 mm to (447.8, 298.0)
- moved U2 1.29 mm to (448.7, 301.2)
- moved C10 1.29 mm to (445.6, 303.0)
- moved C9 1.29 mm to (445.6, 299.7)
- moved R9 0.87 mm to (444.0, 300.3)
Routing:
- net /DAT0: track 0.00 -> 356.7 mm, vias 0 -> 3
- net /DAT1: track 0.00 -> 356.6 mm, vias 0 -> 3
- net /CLK0: track 520.6 -> 519.3 mm

Commit message: data 2,3 routed
Routing:
- net /DAT3: track 0.00 -> 352.0 mm, vias 0 -> 3
- net /DAT2: track 0.00 -> 349.4 mm, vias 0 -> 3
