File: recorder/recorder.kicad_pcb (KiCad board)
At the start: 4 copper layers, 34 parts, among them J1 GPIO_Conn_02x20_Odd_Even, U1 IM73D122V01, U10 TPS7A4700RGWT, U2 ADAU7118, U3 IM73D122V01, U4 IM73D122V01, U5 IM73D122V01, U6 IM73D122V01, U7 IM73D122V01, U8 IM73D122V01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

Commit message: routing progress, dvdd, iovdd, gnd
Routing:
- net GND: track 0.00 -> 57.7 mm, vias 0 -> 29
- net /DVDD: track 29.0 -> 46.0 mm, vias 0 -> 10
- net /IOVDD: track 0.00 -> 10.9 mm
- net /ENABLE: track 0.00 -> 4.59 mm, vias 0 -> 2
- net /DAT2: track 349.4 -> 352.2 mm
- net /DAT1: track 356.6 -> 358.5 mm
- net Net-(U10-NR): track 0.00 -> 1.68 mm

Commit message: pre-move
Parts:
- moved J1 74.8 mm to (497.6, 291.5), turned to -90 degrees
- turned C10 to 90 degrees
Routing:
- net /ENABLE: track 4.59 -> 7.25 mm, vias 2 -> 0
- net /IOVDD: track 10.9 -> 9.93 mm
- net GND: track 57.7 -> 57.0 mm

Commit message: new layout
Parts:
- moved C10 22.5 mm to (423.0, 303.0)
- moved C11 22.5 mm to (425.2, 298.0)
- moved C12 22.5 mm to (419.1, 304.0)
- moved C13 22.5 mm to (416.6, 296.0)
- moved C14 22.5 mm to (416.1, 304.0)
- moved C9 22.5 mm to (423.0, 299.7)
- moved R9 22.5 mm to (421.5, 300.3)
- moved U10 22.5 mm to (417.5, 300.0)
- moved U2 22.5 mm to (426.2, 301.2)
- moved J1 17.6 mm to (481.4, 298.5)
Routing:
- net /IOVDD: track 9.93 -> 78.3 mm, vias 0 -> 1
- net /SCL: track 0.00 -> 23.3 mm, vias 0 -> 1
- net /DAT3: track 352.0 -> 374.5 mm
- net /CLK1: track 515.6 -> 538.2 mm
- net /DAT2: track 352.2 -> 374.8 mm
- net /SDA: track 0.00 -> 21.8 mm, vias 0 -> 1
- net /CLK0: track 519.5 -> 537.2 mm
- net /DAT0: track 356.7 -> 372.9 mm
- net /DAT1: track 358.5 -> 374.5 mm
- net /DIN: track 0.00 -> 12.5 mm

Commit message: routed and traced
Parts:
- moved C11 1.04 mm to (424.5, 297.3), turned to 90 degrees
Routing:
- net /SCLK: track 0.00 -> 47.8 mm, vias 0 -> 2
- net /FS: track 0.00 -> 13.5 mm, vias 0 -> 2
- net /CLK0: track 537.2 -> 543.4 mm
- net /DAT1: track 374.5 -> 370.0 mm
- net /CLK1: track 538.2 -> 542.0 mm
- net /DIN: track 12.5 -> 15.3 mm
- net /DAT3: track 374.5 -> 376.1 mm
- net /SDA: track 21.8 -> 23.1 mm
- net /IOVDD: track 78.3 -> 79.1 mm
