File: recorder/recorder.kicad_sch (KiCad schematic)
At the start: 13 parts, among them J1 GPIO_Conn_02x20_Odd_Even, U10 TPS7A4700RGWT, U2 ADAU7118

Commit message: Polarization check of Capacitors
Parts:
- C10, C11, C9: value 100nF -> 220nF; symbol recorder:C_Small_1 -> recorder:C_220nF; MPN MCASJ168BD7475KTCA01 -> 06036C223KAT2A
- C12: symbol recorder:C_Small_1 -> recorder:C_1uF; MPN MCASJ168BD7475KTCA01 -> 06036C105MAT2A
- C13: value 47uF -> 4700nF; symbol recorder:C_Small_1 -> recorder:C_4700nF
- C14: symbol recorder:C_Small_1 -> recorder:C_10uF; MPN MCASJ168BD7475KTCA01 -> CL10B106MQ8NRNC
- J1: now not fitted
- R12, R13, R14: symbol Device:R -> recorder:R_22; MPN (none) -> ESR03EZPJ220; Package (none) -> 0603 (1608 Metric)
- R9: value 10k0 -> 10000; symbol Device:R -> recorder:R_10000; MPN (none) -> RNCE0603BTE10K0; Package (none) -> 0603 (1608 Metric)
Connections:
- net GND: now also C10.2, C12.2; no longer C10.1, C12.1
- net IOVDD: now also C10.1; no longer C10.2
- net at U10.14 (NR): now also C12.1; no longer C12.2
